Commit message: Add camera link and fix body link coordinates

File: src/rover_description/urdf/rover.urdf.xacro (robot description, xacro)
@@ -7,4 +7,6 @@
     <xacro:include filename="$(find rover_description)/urdf/rover_gazebo.xacro" />
     <xacro:include filename="$(find rover_description)/urdf/rover_control.xacro" />
+    <xacro:include filename="$(find rover_description)/urdf/sensors/realsense.xacro" />
+    <!-- <xacro:include filename="$(find rover_description)/urdf/sensors/imu.xacro" /> -->
     <link name="base_footprint"/>
     <joint name="base_footprint_joint" type="fixed">
@@ -21,5 +23,5 @@
         </inertial>
         <visual>
-            <origin rpy="0 0 1.579795" xyz="0 0.03 0"/>
+            <origin rpy="0 0 1.579795" xyz="0 0 0"/>
             <geometry>
                 <!--<box size="1 0.6 0.3"/>-->
@@ -31,5 +33,5 @@
         </visual>
         <collision>
-            <origin rpy="0 0 1.579795" xyz="0 0.03 0"/>
+            <origin rpy="0 0 1.579795" xyz="0 0 0"/>
             <geometry>
                 <mesh filename="package://rover_description/meshes/base_link.stl" scale="0.001 0.001 0.001" />

Commit message: add camera

File: src/rover_description/urdf/rover.urdf.xacro (robot description, xacro)
@@ -4,8 +4,8 @@
     xmlns:xacro="http://ros.org/wiki/xacro">
     <xacro:arg name="is_sim" default="true" />
-    <xacro:arg name="is_ignition" default="true"/>
+    <xacro:arg name="is_ignition" default="false"/>
+    <!-- <xacro:include filename="$(find rover_description)/urdf/sensors/realsense.xacro" /> -->
+    <xacro:include filename="$(find rover_description)/urdf/rover_control.xacro" />
     <xacro:include filename="$(find rover_description)/urdf/rover_gazebo.xacro" />
-    <xacro:include filename="$(find rover_description)/urdf/rover_control.xacro" />
-    <xacro:include filename="$(find rover_description)/urdf/sensors/realsense.xacro" />
     <!-- <xacro:include filename="$(find rover_description)/urdf/sensors/imu.xacro" /> -->
     <link name="base_footprint"/>
@@ -271,4 +271,36 @@
         </collision>
     </link>
+    <joint name="camera_joint" type="fixed">
+        <parent link="body_link"/>
+        <child link="camera_link"/>
+        <origin xyz="0.56 0.0 0.1" rpy="0.0 0.0 0.0"/>
+        <axis xyz="0 1 0" />
+    </joint>
+    <link name="camera_link">
+        <collision>
+            <geometry>
+                <box size="0.010 0.03 0.03"/>
+            </geometry>
+            <material name="yellow">
+                <color rgba="1 1 0 1"/>
+            </material>
+        </collision>
+        <visual>
+            <geometry>
+                <box size="0.010 0.03 0.03"/>
+            </geometry>
+            <material name="yellow">
+                <color rgba="1 1 0 1"/>
+            </material>
+        </visual>
+    </link>
+    <!-- Optical joint will rotate the camera because it uses a different coordinate system where two axis are inverted -->
+    <joint name="camera_optical_joint" type="fixed">
+        <parent link="camera_link"/>
+        <child link="camera_link_optical"/>
+        <origin xyz="0.01 0.01 0.01" rpy="-1.5707 0 -1.5707"/>
+    </joint>
+    <link name="camera_link_optical">
+    </link>
     <!-- This is the back left wheel of the rover
     <joint name="wheel2_joint" type="continuous">

File: src/rover_description/urdf/rover_gazebo.xacro (robot description, xacro)
@@ -71,3 +71,33 @@
     </xacro:unless>
   </gazebo>
+  <gazebo reference="camera_link">
+    <sensor name="camera" type="camera">
+      <camera>
+        <horizontal_fov>1.3962634</horizontal_fov>
+        <image>
+          <width>640</width>
+          <height>480</height>
+          <format>R8G8B8</format>
+        </image>
+        <clip>
+          <near>0.1</near>
+          <far>15</far>
+        </clip>
+        <noise>
+          <type>gaussian</type>
+          <!-- Noise is sampled independently per pixel on each frame.
+               That pixel's noise value is added to each of its color
+               channels, which at that point lie in the range [0,1]. -->
+          <mean>0.0</mean>
+          <stddev>0.007</stddev>
+        </noise>
+        <optical_frame_id>camera_link_optical</optical_frame_id>
+        <camera_info_topic>camera/camera_info</camera_info_topic>
+      </camera>
+      <always_on>1</always_on>
+      <update_rate>20</update_rate>
+      <visualize>true</visualize>
+      <topic>camera/image</topic>
+    </sensor>
+  </gazebo>
 </robot>

File: src/rover_description/urdf/sensors/realsense.xacro (robot description, xacro)
@@ -2,33 +2,3 @@
 <robot xmlns:xacro="http://ros.org/wiki/xacro">
   <!-- Add realsense stl -->
-  <joint name="realsense_joint" type="fixed">
-    <parent link="body_link"/>
-    <child link="realsense_link"/>
-    <origin xyz="-0.36 0.0 0.08" rpy="0.0 0.0 0.0"/>
-  </joint>
-  <link name="realsense_link">
-    <visual>
-      <geometry>
-        <box size="0.010 0.03 0.03"/>
-      </geometry>
-      <material name="yellow">
-        <color rgba="1 1 0 1"/>
-      </material>
-    </visual>
-  </link>
-  <!-- Optical joint will rotate the camera because it uses a different coordinate system where two axis are inverted -->
-  <joint name="realsense_optical_joint" type="fixed">
-    <parent link="realsense_link"/>
-    <child link="realsense_link_optical"/>
-    <origin xyz="0 0 0" rpy="${-pi/2} 0 ${-pi/2}"/>
-  </joint>
-  <link name="realsense_link_optical">
-  </link>
-  <!-- End of Optical joint -->
-  <!-- <gazebo reference="realsense_link">
-    <material>
-    Gazebo/Red
-    </material>
-  </gazebo> -->
-  <!-- TODO: Add 2d realsense and Depth realsense simulation -->
 </robot>
